Commit message: update model

File: res/ur10_moveit_config/ur10.urdf (robot description, URDF)
Before this commit: robot ur10, 11 links, 10 joints
Links:
- removed link world
- link base_link: geometry collision mesh filename=package://universial_robot_ign/models/ur10/meshes/collision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; visual mesh filename=package://universial_robot_ign/models/ur10/meshes/visual/ba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
- link forearm_link: geometry collision mesh filename=package://universial_robot_ign/models/ur10/meshes/collision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; visual mesh filename=package://universial_robot_ign/models/ur10/meshes/visual/fo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
- link shoulder_link: geometry collision mesh filename=package://universial_robot_ign/models/ur10/meshes/collision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; visual mesh filename=package://universial_robot_ign/models/ur10/meshes/visual/sh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
- link upper_arm_link: geometry collision mesh filename=package://universial_robot_ign/models/ur10/meshes/collision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; visual mesh filename=package://universial_robot_ign/models/ur10/meshes/visual/up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
- link wrist_1_link: geometry collision mesh filename=package://universial_robot_ign/models/ur10/meshes/collision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; visual mesh filename=package://universial_robot_ign/models/ur10/meshes/visual/wr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
- link wrist_2_link: geometry collision mesh filename=package://universial_robot_ign/models/ur10/meshes/collision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; visual mesh filename=package://universial_robot_ign/models/ur10/meshes/visual/wr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
- link wrist_3_link: geometry collision mesh filename=package://universial_robot_ign/models/ur10/meshes/collision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; visual mesh filename=package://universial_robot_ign/models/ur10/meshes/visual/wr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
Joints:
- removed joint world_joint

Commit message: update doc

File: res/ur10_moveit_config/ur10.urdf (robot description, URDF)
Before this commit: robot ur10, 10 links, 9 joints
Links:
- link base_link: geometry collision mesh filename=package://universal_robot_ign/models/ur10/meshes/collision/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; visual mesh filename=package://universal_robot_ign/models/ur10/meshes/visual/bas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
- link forearm_link: geometry collision mesh filename=package://universal_robot_ign/models/ur10/meshes/collision/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; visual mesh filename=package://universal_robot_ign/models/ur10/meshes/visual/for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
- link shoulder_link: geometry collision mesh filename=package://universal_robot_ign/models/ur10/meshes/collision/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; visual mesh filename=package://universal_robot_ign/models/ur10/meshes/visual/sho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
- link upper_arm_link: geometry collision mesh filename=package://universal_robot_ign/models/ur10/meshes/collision/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; visual mesh filename=package://universal_robot_ign/models/ur10/meshes/visual/upp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
- link wrist_1_link: geometry collision mesh filename=package://universal_robot_ign/models/ur10/meshes/collision/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; visual mesh filename=package://universal_robot_ign/models/ur10/meshes/visual/wri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
- link wrist_2_link: geometry collision mesh filename=package://universal_robot_ign/models/ur10/meshes/collision/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; visual mesh filename=package://universal_robot_ign/models/ur10/meshes/visual/wri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
- link wrist_3_link: geometry collision mesh filename=package://universal_robot_ign/models/ur10/meshes/collision/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; visual mesh filename=package://universal_robot_ign/models/ur10/meshes/visual/wri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
