Commit message: update

File: resource/models/ur3/ur3.def.xacro (robot description, xacro)
@@ -3,16 +3,16 @@
     <!--model definition-->
     <!--xacro(https://github.com/ros-industrial/universal_robot) -> urdf(use xacro) -> sdf(use ign sdf -p),and it's modified -->
-    <xacro_define_macro name='ur10' params="parent">
+    <xmacro_define_block name='ur3' params="parent">
         <link name='base_link'>
-            <pose relative_to='${parent}'>0 0 0 0 -0 0</pose>
-            <inertial>
-                <mass>4</mass>
-                <inertia>
-                    <ixx>0.00610633</ixx>
-                    <ixy>0</ixy>
-                    <ixz>0</ixz>
-                    <iyy>0.00610633</iyy>
-                    <iyz>0</iyz>
-                    <izz>0.01125</izz>
+            <pose relative_to='${parent}'>0 0 0 0 0 0</pose>
+            <inertial>
+                <mass>2</mass>
+                <inertia>
+                    <ixx>0.00305317</ixx>
+                    <ixy>0</ixy>
+                    <ixz>0</ixz>
+                    <iyy>0.00305317</iyy>
+                    <iyz>0</iyz>
+                    <izz>0.005625</izz>
                 </inertia>
             </inertial>
@@ -20,5 +20,5 @@
                 <geometry>
                     <mesh>
-                        <uri>model://ur10/meshes/collision/base.stl</uri>
+                        <uri>model://ur3/meshes/collision/base.stl</uri>
                     </mesh>
                 </geometry>
@@ -27,12 +27,11 @@
                 <geometry>
                     <mesh>
-                        <uri>model://ur10/meshes/visual/base.dae</uri>
-                    </mesh>
-                </geometry>
-            </visual>
-            <self_collide>1</self_collide>
+                        <uri>model://ur3/meshes/visual/base.dae</uri>
+                    </mesh>
+                </geometry>
+            </visual>
         </link>
         <joint name='shoulder_pan_joint' type='revolute'>
-            <pose relative_to='base_link'>0 0 0.1273 0 -0 0</pose>
+            <pose relative_to='base_link'>0 0 0.1519 0 -0 0</pose>
             <parent>base_link</parent>
             <child>shoulder_link</child>
@@ -56,12 +55,12 @@
             <pose relative_to='shoulder_pan_joint'>0 0 0 0 -0 0</pose>
             <inertial>
-                <mass>7.778</mass>
-                <inertia>
-                    <ixx>0.0314743</ixx>
-                    <ixy>0</ixy>
-                    <ixz>0</ixz>
-                    <iyy>0.0314743</iyy>
-                    <iyz>0</iyz>
-                    <izz>0.0218756</izz>
+                <mass>2</mass>
+                <inertia>
+                    <ixx>0.00809316</ixx>
+                    <ixy>0</ixy>
+                    <ixz>0</ixz>
+                    <iyy>0.00809316</iyy>
+                    <iyz>0</iyz>
+                    <izz>0.005625</izz>
                 </inertia>
             </inertial>
@@ -69,5 +68,5 @@
                 <geometry>
                     <mesh>
-                        <uri>model://ur10/meshes/collision/shoulder.stl</uri>
+                        <uri>model://ur3/meshes/collision/shoulder.stl</uri>
                     </mesh>
                 </geometry>
@@ -76,5 +75,5 @@
                 <geometry>
                     <mesh>
-                        <uri>model://ur10/meshes/visual/shoulder.dae</uri>
+                        <uri>model://ur3/meshes/visual/shoulder.dae</uri>
                     </mesh>
                 </geometry>
@@ -83,5 +82,5 @@
         </link>
         <joint name='shoulder_lift_joint' type='revolute'>
-            <pose relative_to='shoulder_link'>0 0.220941 0 0 1.5708 0</pose>
+            <pose relative_to='shoulder_link'>0 0.1198 0 0 1.5708 0</pose>
             <parent>shoulder_link</parent>
             <child>upper_arm_link</child>
@@ -105,13 +104,13 @@
             <pose relative_to='shoulder_lift_joint'>0 0 0 0 -0 0</pose>
             <inertial>
-                <pose>0 -0.045 0.306 0 -0 0</pose>
-                <mass>12.93</mass>
-                <inertia>
-                    <ixx>0.421754</ixx>
-                    <ixy>0</ixy>
-                    <ixz>0</ixz>
-                    <iyy>0.421754</iyy>
-                    <iyz>0</iyz>
-                    <izz>0.0363656</izz>
+                <pose>0 0 0.121825 0 -0 0</pose>
+                <mass>3.42</mass>
+                <inertia>
+                    <ixx>0.0217285</ixx>
+                    <ixy>0</ixy>
+                    <ixz>0</ixz>
+                    <iyy>0.0217285</iyy>
+                    <iyz>0</iyz>
+                    <izz>0.00961875</izz>
                 </inertia>
             </inertial>
@@ -119,5 +118,5 @@
                 <geometry>
                     <mesh>
-                        <uri>model://ur10/meshes/collision/upperarm.stl</uri>
+                        <uri>model://ur3/meshes/collision/upperarm.stl</uri>
                     </mesh>
                 </geometry>
@@ -126,5 +125,5 @@
                 <geometry>
                     <mesh>
-                        <uri>model://ur10/meshes/visual/upperarm.dae</uri>
+                        <uri>model://ur3/meshes/visual/upperarm.dae</uri>
                     </mesh>
                 </geometry>
@@ -133,5 +132,5 @@
         </link>
         <joint name='elbow_joint' type='revolute'>
-            <pose relative_to='upper_arm_link'>0 -0.1719 0.612 0 -0 0</pose>
+            <pose relative_to='upper_arm_link'>0 -0.0925 0.24365 0 -0 0</pose>
             <parent>upper_arm_link</parent>
             <child>forearm_link</child>
@@ -155,13 +154,13 @@
             <pose relative_to='elbow_joint'>0 0 0 0 -0 0</pose>
             <inertial>
-                <pose>0 0 0.28615 0 -0 0</pose>
-                <mass>3.87</mass>
-                <inertia>
-                    <ixx>0.11107</ixx>
-                    <ixy>0</ixy>
-                    <ixz>0</ixz>
-                    <iyy>0.11107</iyy>
-                    <iyz>0</iyz>
-                    <izz>0.0108844</izz>
+                <pose>0 0 0.106625 0 -0 0</pose>
+                <mass>1.26</mass>
+                <inertia>
+                    <ixx>0.00654681</ixx>
+                    <ixy>0</ixy>
+                    <ixz>0</ixz>
+                    <iyy>0.00654681</iyy>
+                    <iyz>0</iyz>
+                    <izz>0.00354375</izz>
                 </inertia>
             </inertial>
@@ -169,5 +168,5 @@
                 <geometry>
                     <mesh>
-                        <uri>model://ur10/meshes/collision/forearm.stl</uri>
+                        <uri>model://ur3/meshes/collision/forearm.stl</uri>
                     </mesh>
                 </geometry>
@@ -176,5 +175,5 @@
                 <geometry>
                     <mesh>
-                        <uri>model://ur10/meshes/visual/forearm.dae</uri>
+                        <uri>model://ur3/meshes/visual/forearm.dae</uri>
                     </mesh>
                 </geometry>
@@ -183,5 +182,5 @@
         </link>
         <joint name='wrist_1_joint' type='revolute'>
-            <pose relative_to='forearm_link'>0 0 0.5723 0 1.5708 0</pose>
+            <pose relative_to='forearm_link'>0 0 0.21325 0 1.5708 0</pose>
             <parent>forearm_link</parent>
             <child>wrist_1_link</child>
@@ -205,13 +204,13 @@
             <pose relative_to='wrist_1_joint'>0 0 0 0 -0 0</pose>
             <inertial>
-                <pose>0 0.1149 0 0 -0 0</pose>
-                <mass>1.96</mass>
-                <inertia>
-                    <ixx>0.00510825</ixx>
-                    <ixy>0</ixy>
-                    <ixz>0</ixz>
-                    <iyy>0.00510825</iyy>
-                    <iyz>0</iyz>
-                    <izz>0.0055125</izz>
+                <pose>0 0.08505 0 0 -0 0</pose>
+                <mass>0.8</mass>
+                <inertia>
+                    <ixx>0.002085</ixx>
+                    <ixy>0</ixy>
+                    <ixz>0</ixz>
+                    <iyy>0.002085</iyy>
+                    <iyz>0</iyz>
+                    <izz>0.00225</izz>
                 </inertia>
             </inertial>
@@ -219,5 +218,5 @@
                 <geometry>
                     <mesh>
-                        <uri>model://ur10/meshes/collision/wrist1.stl</uri>
+                        <uri>model://ur3/meshes/collision/wrist1.stl</uri>
                     </mesh>
                 </geometry>
@@ -226,5 +225,5 @@
                 <geometry>
                     <mesh>
-                        <uri>model://ur10/meshes/visual/wrist1.dae</uri>
+                        <uri>model://ur3/meshes/visual/wrist1.dae</uri>
                     </mesh>
                 </geometry>
@@ -233,5 +232,5 @@
         </link>
         <joint name='wrist_2_joint' type='revolute'>
-            <pose relative_to='wrist_1_link'>0 0.1149 0 0 -0 0</pose>
+            <pose relative_to='wrist_1_link'>0 0.08505 0 0 -0 0</pose>
             <parent>wrist_1_link</parent>
             <child>wrist_2_link</child>
@@ -255,13 +254,13 @@
             <pose relative_to='wrist_2_joint'>0 0 0 0 -0 0</pose>
             <inertial>
-                <pose>0 0 0.1157 0 -0 0</pose>
-                <mass>1.96</mass>
-                <inertia>
-                    <ixx>0.00510825</ixx>
-                    <ixy>0</ixy>
-                    <ixz>0</ixz>
-                    <iyy>0.00510825</iyy>
-                    <iyz>0</iyz>
-                    <izz>0.0055125</izz>
+                <pose>0 0 0.08535 0 -0 0</pose>
+                <mass>0.8</mass>
+                <inertia>
+                    <ixx>0.002085</ixx>
+                    <ixy>0</ixy>
+                    <ixz>0</ixz>
+                    <iyy>0.002085</iyy>
+                    <iyz>0</iyz>
+                    <izz>0.00225</izz>
                 </inertia>
             </inertial>
@@ -269,5 +268,5 @@
                 <geometry>
                     <mesh>
-                        <uri>model://ur10/meshes/collision/wrist2.stl</uri>
+                        <uri>model://ur3/meshes/collision/wrist2.stl</uri>
                     </mesh>
                 </geometry>
@@ -276,5 +275,5 @@
                 <geometry>
                     <mesh>
-                        <uri>model://ur10/meshes/visual/wrist2.dae</uri>
+                        <uri>model://ur3/meshes/visual/wrist2.dae</uri>
                     </mesh>
                 </geometry>
@@ -283,5 +282,5 @@
         </link>
         <joint name='wrist_3_joint' type='revolute'>
-            <pose relative_to='wrist_2_link'>0 0 0.1157 0 -0 0</pose>
+            <pose relative_to='wrist_2_link'>0 0 0.08535 0 -0 0</pose>
             <parent>wrist_2_link</parent>
             <child>wrist_3_link</child>
@@ -305,13 +304,13 @@
             <pose relative_to='wrist_3_joint'>0 0 0 0 -0 0</pose>
             <inertial>
-                <pose>0 0.07695 0 1.5708 -0 0</pose>
-                <mass>0.202</mass>
-                <inertia>
-                    <ixx>0.000117922</ixx>
-                    <ixy>0</ixy>
-                    <ixz>0</ixz>
-                    <iyy>0.000117922</iyy>
-                    <iyz>0</iyz>
-                    <izz>0.000204525</izz>
+                <pose>0 0.0619 0 1.5708 -0 0</pose>
+                <mass>0.35</mass>
+                <inertia>
+                    <ixx>0.000136267</ixx>
+                    <ixy>0</ixy>
+                    <ixz>0</ixz>
+                    <iyy>0.000136267</iyy>
+                    <iyz>0</iyz>
+                    <izz>0.0001792</izz>
                 </inertia>
             </inertial>
@@ -319,5 +318,5 @@
                 <geometry>
                     <mesh>
-                        <uri>model://ur10/meshes/collision/wrist3.stl</uri>
+                        <uri>model://ur3/meshes/collision/wrist3.stl</uri>
                     </mesh>
                 </geometry>
@@ -326,10 +325,10 @@
                 <geometry>
                     <mesh>
-                        <uri>model://ur10/meshes/visual/wrist3.dae</uri>
-                    </mesh>
-                </geometry>
-            </visual>
-            <self_collide>1</self_collide>
-        </link>
-    </xacro_define_macro>
+                        <uri>model://ur3/meshes/visual/wrist3.dae</uri>
+                    </mesh>
+                </geometry>
+            </visual>
+            <self_collide>1</self_collide>
+        </link>
+    </xmacro_define_block>
 </sdf>
