Commit message: update

File: resource/models/ur5/ur5.def.xacro (robot description, xacro)
@@ -3,16 +3,16 @@
     <!--model definition-->
     <!--xacro(https://github.com/ros-industrial/universal_robot) -> urdf(use xacro) -> sdf(use ign sdf -p),and it's modified -->
-    <xacro_define_macro name='ur3' params="parent">
+    <xmacro_define_block name='ur5' params="parent">
         <link name='base_link'>
             <pose relative_to='${parent}'>0 0 0 0 0 0</pose>
             <inertial>
-                <mass>2</mass>
-                <inertia>
-                    <ixx>0.00305317</ixx>
-                    <ixy>0</ixy>
-                    <ixz>0</ixz>
-                    <iyy>0.00305317</iyy>
-                    <iyz>0</iyz>
-                    <izz>0.005625</izz>
+                <mass>4</mass>
+                <inertia>
+                    <ixx>0.00443333</ixx>
+                    <ixy>0</ixy>
+                    <ixz>0</ixz>
+                    <iyy>0.00443333</iyy>
+                    <iyz>0</iyz>
+                    <izz>0.0072</izz>
                 </inertia>
             </inertial>
@@ -20,5 +20,5 @@
                 <geometry>
                     <mesh>
-                        <uri>model://ur3/meshes/collision/base.stl</uri>
+                        <uri>model://ur5/meshes/collision/base.stl</uri>
                     </mesh>
                 </geometry>
@@ -27,5 +27,5 @@
                 <geometry>
                     <mesh>
-                        <uri>model://ur3/meshes/visual/base.dae</uri>
+                        <uri>model://ur5/meshes/visual/base.dae</uri>
                     </mesh>
                 </geometry>
@@ -33,5 +33,5 @@
         </link>
         <joint name='shoulder_pan_joint' type='revolute'>
-            <pose relative_to='base_link'>0 0 0.1519 0 -0 0</pose>
+            <pose relative_to='base_link'>0 0 0.089159 0 -0 0</pose>
             <parent>base_link</parent>
             <child>shoulder_link</child>
@@ -41,6 +41,6 @@
                     <lower>-6.28319</lower>
                     <upper>6.28319</upper>
-                    <effort>330</effort>
-                    <velocity>2.16</velocity>
+                    <effort>150</effort>
+                    <velocity>3.15</velocity>
                 </limit>
                 <dynamics>
@@ -55,12 +55,12 @@
             <pose relative_to='shoulder_pan_joint'>0 0 0 0 -0 0</pose>
             <inertial>
-                <mass>2</mass>
-                <inertia>
-                    <ixx>0.00809316</ixx>
-                    <ixy>0</ixy>
-                    <ixz>0</ixz>
-                    <iyy>0.00809316</iyy>
-                    <iyz>0</iyz>
-                    <izz>0.005625</izz>
+                <mass>3.7</mass>
+                <inertia>
+                    <ixx>0.0102675</ixx>
+                    <ixy>0</ixy>
+                    <ixz>0</ixz>
+                    <iyy>0.0102675</iyy>
+                    <iyz>0</iyz>
+                    <izz>0.00666</izz>
                 </inertia>
             </inertial>
@@ -68,5 +68,5 @@
                 <geometry>
                     <mesh>
-                        <uri>model://ur3/meshes/collision/shoulder.stl</uri>
+                        <uri>model://ur5/meshes/collision/shoulder.stl</uri>
                     </mesh>
                 </geometry>
@@ -75,5 +75,5 @@
                 <geometry>
                     <mesh>
-                        <uri>model://ur3/meshes/visual/shoulder.dae</uri>
+                        <uri>model://ur5/meshes/visual/shoulder.dae</uri>
                     </mesh>
                 </geometry>
@@ -82,5 +82,5 @@
         </link>
         <joint name='shoulder_lift_joint' type='revolute'>
-            <pose relative_to='shoulder_link'>0 0.1198 0 0 1.5708 0</pose>
+            <pose relative_to='shoulder_link'>0 0.13585 0 0 1.5708 0</pose>
             <parent>shoulder_link</parent>
             <child>upper_arm_link</child>
@@ -90,6 +90,6 @@
                     <lower>-6.28319</lower>
                     <upper>6.28319</upper>
-                    <effort>330</effort>
-                    <velocity>2.16</velocity>
+                    <effort>150</effort>
+                    <velocity>3.15</velocity>
                 </limit>
                 <dynamics>
@@ -104,13 +104,13 @@
             <pose relative_to='shoulder_lift_joint'>0 0 0 0 -0 0</pose>
             <inertial>
-                <pose>0 0 0.121825 0 -0 0</pose>
-                <mass>3.42</mass>
-                <inertia>
-                    <ixx>0.0217285</ixx>
-                    <ixy>0</ixy>
-                    <ixz>0</ixz>
-                    <iyy>0.0217285</iyy>
-                    <iyz>0</iyz>
-                    <izz>0.00961875</izz>
+                <pose>0 0 0.28 0 -0 0</pose>
+                <mass>8.393</mass>
+                <inertia>
+                    <ixx>0.226891</ixx>
+                    <ixy>0</ixy>
+                    <ixz>0</ixz>
+                    <iyy>0.226891</iyy>
+                    <iyz>0</iyz>
+                    <izz>0.0151074</izz>
                 </inertia>
             </inertial>
@@ -118,5 +118,5 @@
                 <geometry>
                     <mesh>
-                        <uri>model://ur3/meshes/collision/upperarm.stl</uri>
+                        <uri>model://ur5/meshes/collision/upperarm.stl</uri>
                     </mesh>
                 </geometry>
@@ -125,5 +125,5 @@
                 <geometry>
                     <mesh>
-                        <uri>model://ur3/meshes/visual/upperarm.dae</uri>
+                        <uri>model://ur5/meshes/visual/upperarm.dae</uri>
                     </mesh>
                 </geometry>
@@ -132,5 +132,5 @@
         </link>
         <joint name='elbow_joint' type='revolute'>
-            <pose relative_to='upper_arm_link'>0 -0.0925 0.24365 0 -0 0</pose>
+            <pose relative_to='upper_arm_link'>0 -0.1197 0.425 0 -0 0</pose>
             <parent>upper_arm_link</parent>
             <child>forearm_link</child>
@@ -154,13 +154,13 @@
             <pose relative_to='elbow_joint'>0 0 0 0 -0 0</pose>
             <inertial>
-                <pose>0 0 0.106625 0 -0 0</pose>
-                <mass>1.26</mass>
-                <inertia>
-                    <ixx>0.00654681</ixx>
-                    <ixy>0</ixy>
-                    <ixz>0</ixz>
-                    <iyy>0.00654681</iyy>
-                    <iyz>0</iyz>
-                    <izz>0.00354375</izz>
+                <pose>0 0 0.196125 0 -0 0</pose>
+                <mass>2.275</mass>
+                <inertia>
+                    <ixx>0.0312168</ixx>
+                    <ixy>0</ixy>
+                    <ixz>0</ixz>
+                    <iyy>0.0312168</iyy>
+                    <iyz>0</iyz>
+                    <izz>0.004095</izz>
                 </inertia>
             </inertial>
@@ -168,5 +168,5 @@
                 <geometry>
                     <mesh>
-                        <uri>model://ur3/meshes/collision/forearm.stl</uri>
+                        <uri>model://ur5/meshes/collision/forearm.stl</uri>
                     </mesh>
                 </geometry>
@@ -175,5 +175,5 @@
                 <geometry>
                     <mesh>
-                        <uri>model://ur3/meshes/visual/forearm.dae</uri>
+                        <uri>model://ur5/meshes/visual/forearm.dae</uri>
                     </mesh>
                 </geometry>
@@ -182,5 +182,5 @@
         </link>
         <joint name='wrist_1_joint' type='revolute'>
-            <pose relative_to='forearm_link'>0 0 0.21325 0 1.5708 0</pose>
+            <pose relative_to='forearm_link'>0 0 0.39225 0 1.5708 0</pose>
             <parent>forearm_link</parent>
             <child>wrist_1_link</child>
@@ -190,5 +190,5 @@
                     <lower>-6.28319</lower>
                     <upper>6.28319</upper>
-                    <effort>54</effort>
+                    <effort>28</effort>
                     <velocity>3.2</velocity>
                 </limit>
@@ -204,13 +204,13 @@
             <pose relative_to='wrist_1_joint'>0 0 0 0 -0 0</pose>
             <inertial>
-                <pose>0 0.08505 0 0 -0 0</pose>
-                <mass>0.8</mass>
-                <inertia>
-                    <ixx>0.002085</ixx>
-                    <ixy>0</ixy>
-                    <ixz>0</ixz>
-                    <iyy>0.002085</iyy>
-                    <iyz>0</iyz>
-                    <izz>0.00225</izz>
+                <pose>0 0.093 0 0 -0 0</pose>
+                <mass>1.219</mass>
+                <inertia>
+                    <ixx>0.0025599</ixx>
+                    <ixy>0</ixy>
+                    <ixz>0</ixz>
+                    <iyy>0.0025599</iyy>
+                    <iyz>0</iyz>
+                    <izz>0.0021942</izz>
                 </inertia>
             </inertial>
@@ -218,5 +218,5 @@
                 <geometry>
                     <mesh>
-                        <uri>model://ur3/meshes/collision/wrist1.stl</uri>
+                        <uri>model://ur5/meshes/collision/wrist1.stl</uri>
                     </mesh>
                 </geometry>
@@ -225,5 +225,5 @@
                 <geometry>
                     <mesh>
-                        <uri>model://ur3/meshes/visual/wrist1.dae</uri>
+                        <uri>model://ur5/meshes/visual/wrist1.dae</uri>
                     </mesh>
                 </geometry>
@@ -232,5 +232,5 @@
         </link>
         <joint name='wrist_2_joint' type='revolute'>
-            <pose relative_to='wrist_1_link'>0 0.08505 0 0 -0 0</pose>
+            <pose relative_to='wrist_1_link'>0 0.093 0 0 -0 0</pose>
             <parent>wrist_1_link</parent>
             <child>wrist_2_link</child>
@@ -240,5 +240,5 @@
                     <lower>-6.28319</lower>
                     <upper>6.28319</upper>
-                    <effort>54</effort>
+                    <effort>28</effort>
                     <velocity>3.2</velocity>
                 </limit>
@@ -254,13 +254,13 @@
             <pose relative_to='wrist_2_joint'>0 0 0 0 -0 0</pose>
             <inertial>
-                <pose>0 0 0.08535 0 -0 0</pose>
-                <mass>0.8</mass>
-                <inertia>
-                    <ixx>0.002085</ixx>
-                    <ixy>0</ixy>
-                    <ixz>0</ixz>
-                    <iyy>0.002085</iyy>
-                    <iyz>0</iyz>
-                    <izz>0.00225</izz>
+                <pose>0 0 0.09465 0 -0 0</pose>
+                <mass>1.219</mass>
+                <inertia>
+                    <ixx>0.0025599</ixx>
+                    <ixy>0</ixy>
+                    <ixz>0</ixz>
+                    <iyy>0.0025599</iyy>
+                    <iyz>0</iyz>
+                    <izz>0.0021942</izz>
                 </inertia>
             </inertial>
@@ -268,5 +268,5 @@
                 <geometry>
                     <mesh>
-                        <uri>model://ur3/meshes/collision/wrist2.stl</uri>
+                        <uri>model://ur5/meshes/collision/wrist2.stl</uri>
                     </mesh>
                 </geometry>
@@ -275,5 +275,5 @@
                 <geometry>
                     <mesh>
-                        <uri>model://ur3/meshes/visual/wrist2.dae</uri>
+                        <uri>model://ur5/meshes/visual/wrist2.dae</uri>
                     </mesh>
                 </geometry>
@@ -282,5 +282,5 @@
         </link>
         <joint name='wrist_3_joint' type='revolute'>
-            <pose relative_to='wrist_2_link'>0 0 0.08535 0 -0 0</pose>
+            <pose relative_to='wrist_2_link'>0 0 0.09465 0 -0 0</pose>
             <parent>wrist_2_link</parent>
             <child>wrist_3_link</child>
@@ -290,5 +290,5 @@
                     <lower>-6.28319</lower>
                     <upper>6.28319</upper>
-                    <effort>54</effort>
+                    <effort>28</effort>
                     <velocity>3.2</velocity>
                 </limit>
@@ -304,13 +304,13 @@
             <pose relative_to='wrist_3_joint'>0 0 0 0 -0 0</pose>
             <inertial>
-                <pose>0 0.0619 0 1.5708 -0 0</pose>
-                <mass>0.35</mass>
-                <inertia>
-                    <ixx>0.000136267</ixx>
-                    <ixy>0</ixy>
-                    <ixz>0</ixz>
-                    <iyy>0.000136267</iyy>
-                    <iyz>0</iyz>
-                    <izz>0.0001792</izz>
+                <pose>0 0.06505 0 1.5708 -0 0</pose>
+                <mass>0.1879</mass>
+                <inertia>
+                    <ixx>8.46959e-05</ixx>
+                    <ixy>0</ixy>
+                    <ixz>0</ixz>
+                    <iyy>8.46959e-05</iyy>
+                    <iyz>0</iyz>
+                    <izz>0.000132117</izz>
                 </inertia>
             </inertial>
@@ -318,5 +318,5 @@
                 <geometry>
                     <mesh>
-                        <uri>model://ur3/meshes/collision/wrist3.stl</uri>
+                        <uri>model://ur5/meshes/collision/wrist3.stl</uri>
                     </mesh>
                 </geometry>
@@ -325,10 +325,10 @@
                 <geometry>
                     <mesh>
-                        <uri>model://ur3/meshes/visual/wrist3.dae</uri>
-                    </mesh>
-                </geometry>
-            </visual>
-            <self_collide>1</self_collide>
-        </link>
-    </xacro_define_macro>
+                        <uri>model://ur5/meshes/visual/wrist3.dae</uri>
+                    </mesh>
+                </geometry>
+            </visual>
+            <self_collide>1</self_collide>
+        </link>
+    </xmacro_define_block>
 </sdf>

File: resource/urdf/robotiq140.urdf (robot description, URDF)
Before this commit: robot robotiq140, 11 links, 10 joints
Links:
- link left_inner_finger: geometry collision mesh filename=package://universal_robot_ign/resource/models/robotiq140/me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; visual mesh filename=package://universal_robot_ign/resource/models/robotiq140/me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
- link left_inner_knuckle: geometry collision mesh filename=package://universal_robot_ign/resource/models/robotiq140/me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; visual mesh filename=package://universal_robot_ign/resource/models/robotiq140/me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
- link left_outer_finger: geometry collision mesh filename=package://universal_robot_ign/resource/models/robotiq140/me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; visual mesh filename=package://universal_robot_ign/resource/models/robotiq140/me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
- link left_outer_knuckle: geometry collision mesh filename=package://universal_robot_ign/resource/models/robotiq140/me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; visual mesh filename=package://universal_robot_ign/resource/models/robotiq140/me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
- link right_inner_finger: geometry collision mesh filename=package://universal_robot_ign/resource/models/robotiq140/me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; visual mesh filename=package://universal_robot_ign/resource/models/robotiq140/me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
- link right_inner_knuckle: geometry collision mesh filename=package://universal_robot_ign/resource/models/robotiq140/me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; visual mesh filename=package://universal_robot_ign/resource/models/robotiq140/me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
- link right_outer_finger: geometry collision mesh filename=package://universal_robot_ign/resource/models/robotiq140/me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; visual mesh filename=package://universal_robot_ign/resource/models/robotiq140/me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
- link right_outer_knuckle: geometry collision mesh filename=package://universal_robot_ign/resource/models/robotiq140/me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; visual mesh filename=package://universal_robot_ign/resource/models/robotiq140/me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
- link robotiq_arg2f_base_link: geometry collision mesh filename=package://universal_robot_ign/resource/models/robotiq140/me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; visual mesh filename=package://universal_robot_ign/resource/models/robotiq140/me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

File: resource/urdf/ur10.urdf (robot description, URDF)
Before this commit: robot ur10, 10 links, 9 joints
Links:
- link base_link: geometry collision mesh filename=package://universal_robot_ign/resource/models/ur10/meshes/c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; visual mesh filename=package://universal_robot_ign/resource/models/ur10/meshes/v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
- link forearm_link: geometry collision mesh filename=package://universal_robot_ign/resource/models/ur10/meshes/c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; visual mesh filename=package://universal_robot_ign/resource/models/ur10/meshes/v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
- link shoulder_link: geometry collision mesh filename=package://universal_robot_ign/resource/models/ur10/meshes/c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; visual mesh filename=package://universal_robot_ign/resource/models/ur10/meshes/v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
- link upper_arm_link: geometry collision mesh filename=package://universal_robot_ign/resource/models/ur10/meshes/c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; visual mesh filename=package://universal_robot_ign/resource/models/ur10/meshes/v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
- link wrist_1_link: geometry collision mesh filename=package://universal_robot_ign/resource/models/ur10/meshes/c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; visual mesh filename=package://universal_robot_ign/resource/models/ur10/meshes/v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
- link wrist_2_link: geometry collision mesh filename=package://universal_robot_ign/resource/models/ur10/meshes/c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; visual mesh filename=package://universal_robot_ign/resource/models/ur10/meshes/v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
- link wrist_3_link: geometry collision mesh filename=package://universal_robot_ign/resource/models/ur10/meshes/c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; visual mesh filename=package://universal_robot_ign/resource/models/ur10/meshes/v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

File: resource/urdf/ur5.urdf (robot description, URDF)
Before this commit: robot ur5, 10 links, 9 joints
Links:
- link base_link: geometry collision mesh filename=package://universal_robot_ign/resource/models/ur5/meshes/co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; visual mesh filename=package://universal_robot_ign/resource/models/ur5/meshes/vi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
- link forearm_link: geometry collision mesh filename=package://universal_robot_ign/resource/models/ur5/meshes/co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; visual mesh filename=package://universal_robot_ign/resource/models/ur5/meshes/vi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
- link shoulder_link: geometry collision mesh filename=package://universal_robot_ign/resource/models/ur5/meshes/co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; visual mesh filename=package://universal_robot_ign/resource/models/ur5/meshes/vi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
- link upper_arm_link: geometry collision mesh filename=package://universal_robot_ign/resource/models/ur5/meshes/co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; visual mesh filename=package://universal_robot_ign/resource/models/ur5/meshes/vi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
- link wrist_1_link: geometry collision mesh filename=package://universal_robot_ign/resource/models/ur5/meshes/co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; visual mesh filename=package://universal_robot_ign/resource/models/ur5/meshes/vi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
- link wrist_2_link: geometry collision mesh filename=package://universal_robot_ign/resource/models/ur5/meshes/co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; visual mesh filename=package://universal_robot_ign/resource/models/ur5/meshes/vi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
- link wrist_3_link: geometry collision mesh filename=package://universal_robot_ign/resource/models/ur5/meshes/co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; visual mesh filename=package://universal_robot_ign/resource/models/ur5/meshes/vi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
